Commit message: Added ground truth laser

File: urdf/robot_from_sdf.xacro (robot description, xacro)
@@ -173,4 +173,8 @@
   </sensor>
   <sensor name='front_laser' update_rate='20'>
+    <parent link='${robot_namespace}/base_link'/>
+    <origin xyz='0.424 0 0.387' rpy='0 -0 0'/>
+  </sensor>
+  <sensor name='front_laser_truth' update_rate='20'>
     <parent link='${robot_namespace}/base_link'/>
     <origin xyz='0.424 0 0.387' rpy='0 -0 0'/>
